Commit message: Ran simulations for ur10 robot

File: welding_robot2.urdf (robot description, URDF)
Before this commit: robot ur10_welding, 14 links, 13 joints
Links:
- removed link flange
- removed link flange_extension
- removed link ft_frame
- removed link tool0
- added link tcp_link
- added link welding_torch, mass 0.1; collision mesh filename=CAD_files/torch.STL scale=0.001 0.001 0.001; visual mesh filename=CAD_files/torch.STL scale=0.001 0.001 0.001
Joints:
- removed joint flange-tool0
- removed joint tool0-flange_extension
- removed joint wrist_3-flange
- removed joint wrist_3_link-ft_frame
- added joint tcp_joint: type fixed, parent welding_torch, child tcp_link, origin xyz=0.04 0.04 0.435 rpy=0.9 0 0
- added joint torch_joint: type fixed, parent wrist_3_link, child welding_torch, origin xyz=0.04 0.04 0 rpy=0 0 3.14
